File: pcb/I2C mux buffer/I2C mux buffer.kicad_pcb (KiCad board)
At the start: 2 copper layers, 61.5 x 26 mm, 19 parts, among them J1 ToF Chassis, J2 ToF Claw, J3 Raspberry Pi, U1 TCA9548APWR, U2 TCA9617ADGKR

Commit message: pcbs reviewed
Parts:
- added G***: LOGO, lib_luca:fizz-logo, F.Cu at (51.2, 95.2)
- added G***: LOGO, lib_luca:hotdog-taichi, B.Cu at (73.5, 85.0)
- moved C3 0.51 mm to (71.0, 78.8)
- moved C4 0.21 mm to (76.8, 78.8)
Routing:
- net GND: track 137.9 -> 6.91 mm, vias 2 -> 0
- net +3V3: track 152.3 -> 138.5 mm, vias 1 -> 0
- net Net-(J3-Pin_4): track 28.9 -> 30.1 mm
- net Net-(J3-Pin_3): track 29.1 -> 30.1 mm
- added copper zone on B.Cu, net GND
- added copper zone on F.Cu, net GND
Other:
- outline, holes or cut-outs redrawn
- board text added: "I2C Mux + Buffer V1.0 Team 4 - Hot Dawgs"
