File: pcb/magnetic_encoder/magnetic_encoder.kicad_pcb (KiCad board)
At the start: 2 copper layers, 29.9 x 29.9 mm, 9 parts, among them J1 Conn_01x02_Pin, J2 Conn_01x04_Pin

Commit message: pcbs reviewed
Parts:
- added G***: LOGO, lib_luca:fizz-logo, F.Cu at (119.5, 45.0)
Routing:
- net +3.3V: track 37.3 -> 34.7 mm
- net Net-(J2-Pin_1): track 13.8 -> 14.9 mm
Other:
- board text added: "Magnetic Encoder Team 4 Hot Dawgs"
- board text removed: "Magnetic Encoder ENPH 253 2025 Team 4"
