File: pcb/reflectance/reflectance.kicad_pcb (KiCad board)
At the start: 2 copper layers, 96 x 40.5 mm, 32 parts, among them J1 JCT 4pin, J2 JCt 4pin, J3 JCT 4pin, J4 Reflectance Sensor 4, J6 Conn_01x03_Pin, J7 Reflectance Sensor 4, J8 Conn_01x05_Pin, U1 LM311, U2 LM311, U3 LM311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

Commit message: pcbs reviewed
Parts:
- added G***: LOGO, lib_luca:hotdog-reflectance, B.Cu at (156.0, 65.5)
Connections:
- U5 pad 1: unconnected-(U5-GND-Pad1) -> GND
- U5 pad 4: unconnected-(U5-V--Pad4) -> GND
- U5 pad 8: unconnected-(U5-V+-Pad8) -> +5V
Routing:
- net +5V: track 156.1 -> 177.6 mm
- net Net-(J8-Pin_5): track 21.6 -> 23.5 mm
- added copper zone on B.Cu, net GND
Other:
- outline, holes or cut-outs redrawn
- board text added: "Reflectance V1.0 Team 4 Hot Dawgs"
- board text removed: "Reflectance Circuit ENPH 253 2025 Team 4"
