File: pcb/motherboard/motherboard.kicad_sch (KiCad schematic)
At the start: 39 parts, among them J1 B2B-XH-A, J10 B3B-XH-A, J11 B3B-XH-A, J12 B5B-XH-A, J13 B5B-XH-A, J14 B2B-XH-A, J2 B5B-XH-A, J3 B3B-XH-A, J4 B4B-XH-A, J5 B2B-XH-A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

Commit message: more schematics going to happen
Parts:
- removed C2: 0.47uF, Capacitor_THT:CP_Radial_D5.0mm_P2.50mm, symbol Device:C_Polarized_US
- removed J14: B2B-XH-A, Connector_JST:JST_XH_B2B-XH-A_1x02_P2.50mm_Vertical, symbol lib_luca:B2B-XH-A
- removed R10, R11, R8, R9: 100k, Resistor_THT:R_Axial_DIN0309_L9.0mm_D3.2mm_P2.54mm_Vertical, symbol Device:R
- removed R12, R7: 1k, Resistor_THT:R_Axial_DIN0309_L9.0mm_D3.2mm_P2.54mm_Vertical, symbol Device:R
- removed U4: LM311, Package_DIP:DIP-8_W7.62mm_Socket, symbol Comparator:LM311
- added TP5: GPIO20, TestPoint:TestPoint_THTPad_D2.0mm_Drill1.0mm, symbol Connector:TestPoint
- renumbered TP7 to TP5, TP8 to TP6, TP9 to TP7
Connections:
- net SWITCH2: no longer names the net of U1.18 (20)
- net SWITCH2: now also TP5.1
- no-connect marks 5 -> 3
